File: kicad/v2/v2.kicad_pcb (KiCad board)
At the start: 2 copper layers, 110 parts, among them U1 Raspberry_Pi_Pico, U2 Raspberry_Pi_Pico

Commit message: fix: symetry
Parts:
- moved U1 4.11 mm to (169.0, 91.0)
Routing:
- net unconnected-(U2-VSYS-Pad39): track 0.00 -> 56.1 mm
- net unconnected-(U1-VSYS-Pad39): track 0.00 -> 52.5 mm
- net Column 05: track 175.4 -> 154.6 mm
- net unconnected-(U2-GND-Pad18): track 0.00 -> 15.3 mm
- net unconnected-(U1-GND-Pad18): track 0.00 -> 12.5 mm
- net Row 01: track 128.5 -> 124.1 mm
- net Row 00: track 141.6 -> 138.3 mm
- net Row 04: track 76.8 -> 74.4 mm
- net Column 04: track 190.0 -> 188.0 mm
- net Row 03: track 150.5 -> 148.7 mm
- net Column 02: track 164.7 -> 163.3 mm
- net Column 03: track 205.3 -> 203.8 mm
- net Column 01: track 187.6 -> 186.7 mm
- net Column 00: track 204.2 -> 203.3 mm
- net Row 02: track 134.5 -> 133.8 mm

Commit message: add: 3.5mm jacks with very messy wiring
Parts:
- added U3: ~, flosLibrary:Lumberg 1503 29 Klinken-Einbaubuchse, F.Cu at (168.3, 164.8)
- added U5: ~, flosLibrary:Lumberg 1503 29 Klinken-Einbaubuchse, F.Cu at (232.0, 164.8)
- moved D34 51.6 mm to (338.0, 138.6)
- moved D35 51.6 mm to (320.0, 138.6)
- moved D38 51.6 mm to (266.0, 128.6)
- moved D39 51.6 mm to (248.0, 133.6)
- moved D40 51.6 mm to (338.0, 155.6)
- moved D41 51.6 mm to (320.0, 155.6)
- moved D42 51.6 mm to (302.0, 140.6)
- moved D43 51.6 mm to (284.0, 135.6)
- moved D44 51.6 mm to (266.0, 145.6)
- moved D45 51.6 mm to (248.0, 150.6)
- moved D46 51.6 mm to (338.0, 172.6)
- moved D47 51.6 mm to (320.0, 172.6)
- moved D48 51.6 mm to (302.0, 157.6)
- moved D49 51.6 mm to (284.0, 152.6)
- moved D50 51.6 mm to (266.0, 162.6)
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Connections:
- U1 pad 38: unconnected-(U1-GND-Pad38) -> Net-(U3-3c)
- U1 pad 39: unconnected-(U1-VSYS-Pad39) -> Net-(U1-VSYS)
- U2 pad 38: unconnected-(U2-GND-Pad38) -> Net-(U5-3c)
- U2 pad 39: unconnected-(U2-VSYS-Pad39) -> Net-(U2-VSYS)
Routing:
- net Row 10: track 194.6 -> 117.3 mm
- net Column 12: track 220.4 -> 293.3 mm
- net Net-(U3-3c): track 0.00 -> 62.4 mm
- net Net-(U1-VSYS): track 0.00 -> 58.9 mm
- net unconnected-(U2-VSYS-Pad39): track 56.1 -> 0.00 mm
- net Row 11: track 184.1 -> 128.5 mm
- net unconnected-(U1-VSYS-Pad39): track 52.5 -> 0.00 mm
- net Column 15: track 242.3 -> 200.1 mm
- net Column 11: track 197.5 -> 161.8 mm
- net Column 10: track 178.4 -> 145.2 mm
- net Row 14: track 119.1 -> 88.8 mm
- net Column 02: track 163.3 -> 133.3 mm
- net Row 12: track 173.4 -> 145.6 mm
- net Net-(U2-VSYS): track 0.00 -> 25.5 mm
- net Column 01: track 186.7 -> 161.2 mm
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Other:
- board outline added: 10 x 3 mm

Commit message: add: finishing touches
Parts:
- added G***: LOGO, LOGO, F.Cu at (296.0, 168.8)
- added G***: LOGO, LOGO, F.Cu at (104.0, 168.8)
- moved D52 6.75 mm to (215.5, 182.3), turned to -150 degrees
Routing:
- net Column 12: track 293.3 -> 176.2 mm
- net Column 13: track 208.1 -> 139.9 mm
- net Column 14: track 211.1 -> 167.7 mm
- net Column 03: track 218.9 -> 178.7 mm
- net Column 15: track 200.1 -> 184.5 mm
- net Column 01: track 161.2 -> 172.2 mm
- net Column 02: track 133.3 -> 143.9 mm
- net Row 13: track 165.4 -> 158.1 mm
- net Net-(D52-A): track 6.41 -> 13.3 mm
- net Column 11: track 161.8 -> 155.9 mm
- net Row 02: track 126.8 -> 123.9 mm
- net Column 04: track 163.3 -> 160.4 mm
- net Row 14: track 88.8 -> 86.5 mm
- net Column 05: track 149.0 -> 147.1 mm
- net Column 10: track 145.2 -> 147.1 mm
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Other:
- board size 10 x 3 mm -> 314.8 x 118.8 mm
- board text added: "Splashboard made with <3 by Flo"
